File: pcb/mpe32board/sensors.kicad_sch (KiCad schematic)
At the start: 88 parts, among them J44 Conn_01x05, U4 TCA9548ARGER, U5 TCA9548ARGER, U6 TCA9548ARGER, U7 TCA9548ARGER, U8 TCA9548ARGER

Commit message: production file changes + ide setup
Parts:
- J44: MPN (none) -> 1719710005
- R10, R11, R12, R13, R14, R15, R16, R17, R18, R19, R20, R25, R26, R27, R28, R29, R30, R31, R32, R33, R34, R35, R36, R37, R38, R39, R40, R43, R44, R45, R46, R47, R48, R49, R5, R50, R51, R52, R53, R54, R55, R56, R57, R58, R6, R61, R62, R63, R64, R65, R66, R67, R68, R69, R7, R70, R71, R72, R73, R74, R75, R76, R79, R8, R80, R81, R82, R83, R84, R85, R86, R87, R88, R89, R9, R90, R91, R92, R93, R94: MPN (none) -> 2.2k 0603
- R23, R24: MPN (none) -> 10k 0603
- U4, U5, U6, U7, U8: MPN (none) -> TCA9548ARGER
