File: pcb/mpe32board/audioic.kicad_sch (KiCad schematic)
At the start: 13 parts, among them J49 AudioJack3_SwitchT, U1 TAC5212IRGER

Commit message: production file changes + ide setup
Parts:
- C26, C30, C32: MPN (none) -> 10uF 1206 X7R
- C27, C29, C31: MPN (none) -> 0.1uF 0603 X7R
- C28: MPN (none) -> 1uF 0603 X7R
- C33, C34: MPN (none) -> 47uF 0603 X7R
- J49: MPN (none) -> SJ-3524-SMT-TR
- R41, R42: MPN (none) -> 1k 0603
- U1: MPN (none) -> TAC5212IRGER
Changed lines of the file:
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@@
+			)
+		)
+		(property "MPN" "10uF 1206 X7R"
+			(at 191.77 58.42 90)
+			(hide yes)
+			(show_name no)
+			(do_not_autoplace no)
+			(effects
+				(font
+					(size 1.27 1.27)
+				)
 			)
 		)
@@
 			)
 		)
+		(property "MPN" "0.1uF 0603 X7R"
+			(at 167.64 48.26 90)
+			(hide yes)
+			(show_name no)
+			(do_not_autoplace no)
+			(effects
+				(font
+					(size 1.27 1.27)
+				)
+			)
+		)
 		(pin "2"
 		)
@@
 			)
 		)
+		(property "MPN" "0.1uF 0603 X7R"
+			(at 123.19 46.99 90)
+			(hide yes)
+			(show_name no)
+			(do_not_autoplace no)
+			(effects
+				(font
+					(size 1.27 1.27)
+				)
+			)
+		)
 		(pin "2"
 		)
@@
 			)
 		)
+		(property "MPN" "1uF 0603 X7R"
+			(at 143.51 57.15 90)
+			(hide yes)
+			(show_name no)
+			(do_not_autoplace no)
+			(effects
+				(font
+					(size 1.27 1.27)
+				)
+			)
+		)
 		(pin "2"
 		)
@@
 			)
 		)
+		(property "MPN" "  SJ-3524-SMT-TR"
+			(at 231.14 78.74 0)
+			(hide yes)
+			(show_name no)
+			(do_not_autoplace no)
+			(effects
+				(font
+					(size 1.27 1.27)
+				)
+			)
+		)
 		(pin "T"
 		)
@@
 			)
 		)
+		(property "MPN" "1k 0603"
+			(at 93.98 107.95 90)
+			(hide yes)
+			(show_name no)
+			(do_not_autoplace no)
+			(effects
+				(font
+					(size 1.27 1.27)
+				)
+			)
+		)
 		(pin "1"
 		)
@@
 		(property "Description" "Polarized capacitor, small symbol"
 			(at 196.85 102.87 0)
+			(hide yes)
+			(show_name no)
+			(do_not_autoplace no)
+			(effects
+				(font
+					(size 1.27 1.27)
+				)
+			)
+		)
+		(property "MPN" "47uF 0603 X7R"
+			(at 196.85 102.87 90)
 			(hide yes)
 			(show_name no)
@@
 			)
 		)
+		(property "MPN" "10uF 1206 X7R"
+			(at 167.64 58.42 90)
+			(hide yes)
+			(show_name no)
+			(do_not_autoplace no)
+			(effects
+				(font
+					(size 1.27 1.27)
+				)
+			)
+		)
 		(pin "2"
 		)
@@
 			)
 		)
+		(property "MPN" "TAC5212IRGER"
+			(at 129.54 80.01 0)
+			(hide yes)
+			(show_name no)
+			(do_not_autoplace no)
+			(effects
+				(font
+					(size 1.27 1.27)
+				)
+			)
+		)
 		(pin "7"
 		)
@@
 			)
 		)
+		(property "MPN" "1k 0603"
+			(at 93.98 100.33 90)
+			(hide yes)
+			(show_name no)
+			(do_not_autoplace no)
+			(effects
+				(font
+					(size 1.27 1.27)
+				)
+			)
+		)
 		(pin "1"
 		)
@@
 			)
 		)
+		(property "MPN" "10uF 1206 X7R"
+			(at 123.19 57.15 90)
+			(hide yes)
+			(show_name no)
+			(do_not_autoplace no)
+			(effects
+				(font
+					(size 1.27 1.27)
+				)
+			)
+		)
 		(pin "2"
 		)
@@
 			)
 		)
+		(property "MPN" "47uF 0603 X7R"
+			(at 201.93 100.33 90)
+			(hide yes)
+			(show_name no)
+			(do_not_autoplace no)
+			(effects
+				(font
+					(size 1.27 1.27)
+				)
+			)
+		)
 		(pin "1"
 		)
@@
 			(hide yes)
 			(show_name no)
+			(do_not_autoplace no)
+			(effects
+				(font
+					(size 1.27 1.27)
+				)
+			)
+		)
+		(property "MPN" "0.1uF 0603 X7R"
+			(at 191.77 48.26 90)
+			(hide yes)
+			(show_name no)
