File: pcb/mpe32board/lcddisplay.kicad_sch (KiCad schematic)
At the start: 7 parts, among them J45 Conn_01x04_Socket, Q1 BSS138, Q2 BSS138

Commit message: production file changes + ide setup
Parts:
- J45: MPN (none) -> DNP
- Q1, Q2: MPN (none) -> BSS138
- R100, R101, R21, R22: MPN (none) -> 10k 0603
Changed lines of the file:
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@@
+			)
+		)
+		(property "MPN" "DNP"
+			(at 144.78 85.09 0)
+			(hide yes)
+			(show_name no)
+			(do_not_autoplace no)
+			(effects
+				(font
+					(size 1.27 1.27)
+				)
 			)
 		)
@@
 			)
 		)
+		(property "MPN" "10k 0603"
+			(at 228.6 102.87 90)
+			(hide yes)
+			(show_name no)
+			(do_not_autoplace no)
+			(effects
+				(font
+					(size 1.27 1.27)
+				)
+			)
+		)
 		(pin "2"
 		)
@@
 		(property "Description" "Resistor, small symbol"
 			(at 246.38 80.01 0)
+			(hide yes)
+			(show_name no)
+			(do_not_autoplace no)
+			(effects
+				(font
+					(size 1.27 1.27)
+				)
+			)
+		)
+		(property "MPN" "10k 0603"
+			(at 246.38 80.01 90)
 			(hide yes)
 			(show_name no)
@@
 			)
 		)
+		(property "MPN" "BSS138"
+			(at 237.49 82.55 90)
+			(hide yes)
+			(show_name no)
+			(do_not_autoplace no)
+			(effects
+				(font
+					(size 1.27 1.27)
+				)
+			)
+		)
 		(pin "1"
 		)
@@
 		(property "Description" "Resistor, small symbol"
 			(at 246.38 102.87 0)
+			(hide yes)
+			(show_name no)
+			(do_not_autoplace no)
+			(effects
+				(font
+					(size 1.27 1.27)
+				)
+			)
+		)
+		(property "MPN" "10k 0603"
+			(at 246.38 102.87 90)
 			(hide yes)
 			(show_name no)
@@
 			)
 		)
+		(property "MPN" "BSS138"
+			(at 237.49 105.41 90)
+			(hide yes)
+			(show_name no)
+			(do_not_autoplace no)
+			(effects
+				(font
+					(size 1.27 1.27)
+				)
+			)
+		)
 		(pin "1"
 		)
@@
 			(hide yes)
 			(show_name no)
+			(do_not_autoplace no)
+			(effects
+				(font
+					(size 1.27 1.27)
+				)
+			)
+		)
+		(property "MPN" "10k 0603"
+			(at 228.6 80.01 90)
+			(hide yes)
+			(show_name no)
