File: pcb/mpe32board/microsd.kicad_sch (KiCad schematic)
At the start: 6 parts, among them J48 Micro_SD_Card_Det_Hirose_DM3AT

Commit message: production file changes + ide setup
Parts:
- J48: MPN (none) -> DM3D-SF
- R95, R96, R97, R98, R99: MPN (none) -> 47k 0603
Changed lines of the file:
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@@
+			)
+		)
+		(property "MPN" "47k 0603"
+			(at 146.05 86.36 0)
+			(hide yes)
+			(show_name no)
+			(do_not_autoplace no)
+			(effects
+				(font
+					(size 1.27 1.27)
+				)
 			)
 		)
@@
 		)
 		(property "Description" "Resistor, small symbol"
+			(at 130.81 86.36 0)
+			(hide yes)
+			(show_name no)
+			(do_not_autoplace no)
+			(effects
+				(font
+					(size 1.27 1.27)
+				)
+			)
+		)
+		(property "MPN" "47k 0603"
 			(at 130.81 86.36 0)
 			(hide yes)
@@
 			)
 		)
+		(property "MPN" "47k 0603"
+			(at 123.19 86.36 0)
+			(hide yes)
+			(show_name no)
+			(do_not_autoplace no)
+			(effects
+				(font
+					(size 1.27 1.27)
+				)
+			)
+		)
 		(pin "2"
 		)
@@
 			)
 		)
+		(property "MPN" "DM3D-SF"
+			(at 198.12 104.14 0)
+			(hide yes)
+			(show_name no)
+			(do_not_autoplace no)
+			(effects
+				(font
+					(size 1.27 1.27)
+				)
+			)
+		)
 		(pin "3"
 		)
@@
 			)
 		)
+		(property "MPN" "47k 0603"
+			(at 138.43 86.36 0)
+			(hide yes)
+			(show_name no)
+			(do_not_autoplace no)
+			(effects
+				(font
+					(size 1.27 1.27)
+				)
+			)
+		)
 		(pin "2"
 		)
@@
 			(at 153.67 86.36 0)
 			(hide yes)
+			(show_name no)
+			(do_not_autoplace no)
+			(effects
+				(font
+					(size 1.27 1.27)
+				)
+			)
+		)
+		(property "MPN" "47k 0603"
+			(at 153.67 86.36 0)
+			(hide yes)
