File: pcb/mpe32board/mpe32board.kicad_sch (KiCad schematic)
At the start: 49 parts, among them J1 Conn_ST_STDC14, J2 USB_C_Receptacle_USB2.0_16P, J46 Conn_02x10_Counter_Clockwise, SW1 SW_Push, SW2 SW_Push, U10 W9812G6KH-75, U11 LM1117MP-3.3, U2 USBLC6-2P6, U9 STM32H743IITx

Commit message: production file changes + ide setup
Parts:
- C1, C42: MPN (none) -> 10uF 1206 X7R
- C10, C11, C12, C13, C14, C17, C2, C22, C23, C24, C25, C3, C35, C36, C37, C38, C39, C4, C40, C41, C5, C6, C7, C8, C9: MPN (none) -> 100nF 0603 X7R
- C15, C16: MPN (none) -> 2.2uF 0603 X7R
- C21, C43: MPN (none) -> 1uF 0603 X7R
- D1: MPN (none) -> SS14
- H1, H2, H3, H4, J46, SW1, SW2: MPN (none) -> DNP
- J1: MPN (none) -> FTSH-107-01-F-DV-K-P-TR
- J2: MPN (none) -> USB4105-GF-A
- R1, R2: MPN (none) -> 10k 0603
- R3, R4: MPN (none) -> 5.1k 0603
- U10: MPN (none) -> W9812G6KH-75
- U11: MPN (none) -> LM1117MP-3.3
- U2: MPN (none) -> USBLC6-2P6
- U9: MPN (none) -> STM32H743IIT
